File: PCB/Dragonfly/Dragonfly.kicad_sch (KiCad schematic)
At the start: 55 parts, among them J1 Conn_01x04_Pin, J2 Micro_SD_Card, Q1 Q_NMOS_GDS, SW1 SW_SPST, SW2 SW_SPST, U1 STM32F405RGTx, U2 ICM-20602, U3 AT32F421G8U7, U4 FD6288Q, X1 TSX-3225

Commit message: updated
Parts:
- added C24, C25, C26, C27, C29, C30: C, symbol Device:C
- added D3, D4, D5: 1N914WT, Diode_SMD:D_SOD-523, symbol Diode:1N914WT
- added J3: Conn_01x02_Pin, symbol Connector:Conn_01x02_Pin
- added Q2, Q3, Q4, Q5, Q6: Q_NMOS_GDS, symbol Transistor_FET:Q_NMOS_GDS
- added R19, R20, R21, R23, R24, R25: 20R, symbol Device:R
- added R22, R26: R, symbol Device:R
- R18: value 20R -> R
Connections:
- net ESC2 A1 is gone; now on net ESC2_A1: R17.1
- net ESC2 B1 is gone; now on net ESC2_B1: R16.1
- net ESC2_l031 is gone; now on net GND: R18.2
- net +8V: now also D3.2 (A), D4.2 (A), D5.2 (A)
- net ESC2 C1: now also Q1.2 (D), U4.12 (VS3), C24.2, Q2.3 (S); no longer R15.1
- net ESC2_H011: now also R25.2
- net ESC2_H021: now also R23.2
- net ESC2_H031: now also R20.2
- net ESC2_L031: now also R19.1
- net GND: now also C27.2, C29.2, C30.2, R22.2, R26.2; no longer Q1.1 (G), Q1.3 (S), R18.1
- net SWCLK1: now also J3.1 (Pin_1)
- net SWDIO1: now also J3.2 (Pin_2)
- net VB3: now reaches U4.14 (VB3)
- net VB3: now also C24.1, C26.1, D3.1 (K), D5.1 (K)
- net ESC2_B1: now reaches U4.15 (VS2)
- net ESC2_B1: now also C25.2, Q3.2 (D), Q4.3 (S)
- net VB2: now reaches U4.17 (VB2)
- net VB2: now also C25.1, D4.1 (K)
- net ESC2_A1: now reaches U4.18 (VS1)
- net ESC2_A1: now also C26.2, Q5.2 (D), Q6.3 (S)
- new net: Q1.3 (S), R18.1
- new net: C27.1, C29.1, C30.1
- new net: Q3.1 (G), R21.1
- new net: Q6.1 (G), R25.1
- new net: Q3.3 (S), R22.1
- new net: Q2.1 (G), R20.1
- new net: Q1.1 (G), R19.2
- new net: Q5.3 (S), R26.1
- new net: Q4.1 (G), R23.1
- new net: Q5.1 (G), R24.1
- new net ESC2_C1: R15.1
- new net ESC2_l011: R24.2
- new net ESC2_l021: R21.2
- new net VIN: Q2.2 (D), Q4.2 (D), Q6.2 (D)
Other:
- moved on the sheet: C21, C22, Q1, R10, R11, R12, R13, R14, R15, R16, R17, R7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

Commit message: Update Dragonfly.kicad_sch
Parts:
- added C28, C31, C33, C37, C38, C39, C40, C42, C46, C47, C48, C49, C51, C55, C56: 10uf, symbol Device:C
- added C32, C34, C35, C36, C41, C43, C44, C45, C50, C52, C53, C54: 100nf, symbol Device:C
- added D10, D11, D12, D13, D14, D6, D7, D8, D9: 1N914WT, Diode_SMD:D_SOD-523, symbol Diode:1N914WT
- added J4, J5, J6: Conn_01x02_Pin, symbol Connector:Conn_01x02_Pin
- added Q10, Q11, Q12, Q13, Q14, Q15, Q16, Q17, Q18, Q19, Q20, Q21, Q22, Q23, Q24, Q7, Q8, Q9: Q_NMOS_GDS, symbol Transistor_FET:Q_NMOS_GDS
- added R27, R28, R29, R33, R34, R35, R36, R37, R42, R44, R46, R47, R48, R49, R53, R54, R55, R56, R57, R62, R64, R66, R67, R68, R69, R73, R74, R75, R76, R77, R82, R84, R86: 10k, symbol Device:R
- added R30, R31, R32, R50, R51, R52, R70, R71, R72: 1k, symbol Device:R
- added R38, R39, R40, R41, R43, R45, R58, R59, R60, R61, R63, R65, R78, R79, R80, R81, R83, R85: 20R, symbol Device:R
- added U10, U6, U8: FD6288Q, QFN50P400X400X90-25N, symbol FD6288Q:FD6288Q
- added U5, U7, U9: AT32F421G8U7, AT32F421G8U7:AT32F421G8U7, symbol AT32F421G8U7:AT32F421G8U7
- C23, C26: value C -> 100nf
- C24, C25, C27, C29, C30: value C -> 10uf
- R1: value 10kΩ NC -> 10k NC
- R10, R11, R15, R16, R17, R18, R22, R26, R9: value R -> 10k
- R12, R13, R14: value R -> 1k
- R2, R3: value 10kΩ -> 10k
- R6: value R -> 0R
Connections:
- net +8V: now also C35.2, C44.2, C53.2, D10.2 (A), D11.2 (A), D12.2 (A), D13.2 (A), D14.2 (A), D6.2 (A), D7.2 (A), D8.2 (A), D9.2 (A), U10.4 (VCC), U6.4 (VCC), U8.4 (VCC)
- net GND: now also Q1.1 (G), Q3.1 (G), Q5.1 (G), R19.2, R21.1, R24.1, C28.2, C31.2, C32.1, C33.2, C34.2, C35.1, C39.2, C40.2, C41.1, C42.2, C43.2, C44.1, C48.2, C49.2, C50.1, C51.2, C52.2, C53.1, Q11.1 (G), Q13.1 (G), Q15.1 (G), Q17.1 (G), Q19.1 (G), Q21.1 (G), Q23.1 (G), Q7.1 (G), Q9.1 (G), R30.1, R31.1, R32.1, R36.1, R38.1, R39.2, R40.1, R42.2, R44.2, R46.2, R50.1, R51.1, R52.1, R56.1, R58.1, R59.2, R60.1, R62.2, R64.2, R66.2, R70.1, R71.1, R72.1, R76.1, R78.1, R79.2, R80.1, R82.2, R84.2, R86.2, U10.6 (COM), U5.16 (VSS), U5.29 (VSS), U6.6 (COM), U7.16 (VSS), U7.29 (VSS), U8.6 (COM), U9.16 (VSS), U9.29 (VSS)
- net VDD33: now also C32.2, C34.1, C41.2, C43.1, C50.2, C52.1, R37.1, R57.1, R77.1, U5.17 (VDD), U5.5 (VDDA), U7.17 (VDD), U7.5 (VDDA), U9.17 (VDD), U9.5 (VDDA)
- net VIN: now also C27.1, C29.1, C30.1, C28.1, C31.1, C33.1, C39.1, C40.1, C42.1, C48.1, C49.1, C51.1, Q10.2 (D), Q12.2 (D), Q14.2 (D), Q16.2 (D), Q18.2 (D), Q20.2 (D), Q22.2 (D), Q24.2 (D), Q8.2 (D)
- net at U4.20 (VB1): now also C26.1, D5.1 (K)
- net VB2: no longer names the net of C25.1, D4.1 (K), U4.17 (VB2)
- net VB3: no longer names the net of C24.1, D3.1 (K), U4.14 (VB3)
- net VB3: no longer C26.1, D5.1 (K)
- new net: R68.2, R72.2, R74.1, U9.10 (PA4)
- new net: R73.2, R74.2, R75.2, U9.7 (PA1)
- new net: Q23.3 (S), R86.1
- new net: Q15.3 (S), R64.1
- new net: Q20.1 (G), R81.1
- new net: R27.2, R31.2, R33.1, U5.11 (PA5)
- new net: C54.1, D12.1 (K), U10.20 (VB1)
- new net: Q18.1 (G), R65.1
- new net: R67.2, R71.2, R73.1, U9.11 (PA5)
- new net: C46.1, D10.1 (K), U8.14 (VB3)
- new net: C47.1, D11.1 (K), U8.17 (VB2)
- new net: C45.1, D9.1 (K), U8.20 (VB1)
- new net: Q8.1 (G), R41.1
- new net: C56.1, D14.1 (K), U10.17 (VB2)
- new net: Q24.1 (G), R85.1
- new net: Q7.3 (S), R42.1
- new net: R28.2, R32.2, R34.1, U5.10 (PA4)
- new net: C36.1, D6.1 (K), U6.20 (VB1)
- new net: Q19.3 (S), R82.1
- new net: Q21.3 (S), R84.1
- new net: C55.1, D13.1 (K), U10.14 (VB3)
- new net: R56.2, U7.1 (BOOT0)
- new net: R29.2, R30.2, R35.1, U5.6 (PA0)
- new net: Q16.1 (G), R63.1
- new net: R76.2, U9.1 (BOOT0)
- new net: C37.1, D7.1 (K), U6.14 (VB3)
- new net: Q9.3 (S), R44.1
- new net: Q17.3 (S), R66.1
- new net: R33.2, R34.2, R35.2, U5.7 (PA1)
- new net: R77.2, U9.4 (NRST)
- new net: C38.1, D8.1 (K), U6.17 (VB2)
- new net: R69.2, R70.2, R75.1, U9.6 (PA0)
- new net: R57.2, U7.4 (NRST)
- new net: R49.2, R50.2, R55.1, U7.6 (PA0)
- new net: R53.2, R54.2, R55.2, U7.7 (PA1)
- new net: R48.2, R52.2, R54.1, U7.10 (PA4)
- new net: R47.2, R51.2, R53.1, U7.11 (PA5)
- new net: Q10.1 (G), R43.1
- new net: R37.2, U5.4 (NRST)
- new net: R36.2, U5.1 (BOOT0)
- new net: Q13.3 (S), R62.1
- new net: Q11.3 (S), R46.1
- new net: Q14.1 (G), R61.1
- new net: Q22.1 (G), R83.1
- new net: Q12.1 (G), R45.1
- new net ESC2 C2: C37.2, C55.2, Q10.3 (S), Q21.2 (D), Q22.3 (S), Q9.2 (D), U10.12 (VS3), U6.12 (VS3)
- new net ESC2 C3: C46.2, Q15.2 (D), Q16.3 (S), U8.12 (VS3)
- new net ESC2_A2: C36.2, C54.2, Q19.2 (D), Q20.3 (S), Q7.2 (D), Q8.3 (S), R29.1, U10.18 (VS1), U6.18 (VS1)
- new net ESC2_A3: C45.2, Q13.2 (D), Q14.3 (S), R49.1, U8.18 (VS1)
- new net ESC2_A4: R69.1
- new net ESC2_B2: C38.2, C56.2, Q11.2 (D), Q12.3 (S), Q23.2 (D), Q24.3 (S), R28.1, U10.15 (VS2), U6.15 (VS2)
- new net ESC2_B3: C47.2, Q17.2 (D), Q18.3 (S), R48.1, U8.15 (VS2)
- new net ESC2_B4: R68.1
- new net ESC2_C2: R27.1
- new net ESC2_C3: R47.1
- new net ESC2_C4: R67.1
- new net ESC2_H012: R41.2, R81.2, U10.19 (HO1), U6.19 (HO1)
- new net ESC2_H013: R61.2, U8.19 (HO1)
- new net ESC2_H022: R45.2, R85.2, U10.16 (HO2), U6.16 (HO2)
- new net ESC2_H023: R65.2, U8.16 (HO2)
- new net ESC2_H032: R43.2, R83.2, U10.13 (HO3), U6.13 (HO3)
- new net ESC2_H033: R63.2, U8.13 (HO3)
- new net ESC2_L012: U10.11 (LO1), U6.11 (LO1)
- new net ESC2_L013: U8.11 (LO1)
- new net ESC2_L022: U10.10 (LO2), U6.10 (LO2)
- new net ESC2_L023: U8.10 (LO2)
- new net ESC2_L032: R39.1, R79.1, U10.9 (LO3), U6.9 (LO3)
- new net ESC2_L033: R59.1, U8.9 (LO3)
- new net ESC2_l012: R38.2, R78.2
- new net ESC2_l013: R58.2
- new net ESC2_l022: R40.2, R80.2
- new net ESC2_l023: R60.2
- new net HI12: U10.22 (HIN1), U5.20 (PA10), U6.22 (HIN1)
- new net HI13: U7.20 (PA10), U8.22 (HIN1)
- new net HI14: U9.20 (PA10)
- new net HI22: U10.23 (HIN2), U5.19 (PA9), U6.23 (HIN2)
- new net HI23: U7.19 (PA9), U8.23 (HIN2)
- new net HI24: U9.19 (PA9)
- new net HI32: U10.24 (HIN3), U5.18 (PA8), U6.24 (HIN3)
- new net HI33: U7.18 (PA8), U8.24 (HIN3)
- new net HI34: U9.18 (PA8)
- new net LI12: U10.1 (LIN1), U5.15 (PB1), U6.1 (LIN1)
- new net LI13: U7.15 (PB1), U8.1 (LIN1)
- new net LI14: U9.15 (PB1)
- new net LI22: U10.2 (LIN2), U5.14 (PB0), U6.2 (LIN2)
- new net LI23: U7.14 (PB0), U8.2 (LIN2)
- new net LI24: U9.14 (PB0)
- new net LI32: U10.3 (LIN3), U5.13 (PA7), U6.3 (LIN3)
- new net LI33: U7.13 (PA7), U8.3 (LIN3)
- new net LI34: U9.13 (PA7)
- new net PWM2: U5.8 (PA2)
- new net PWM3: U7.8 (PA2)
- new net PWM4: U9.8 (PA2)
- new net SWCLK2: J4.1 (Pin_1), U5.22 (PA14)
- new net SWCLK3: J5.1 (Pin_1), J6.1 (Pin_1), U7.22 (PA14)
- new net SWCLK4: U9.22 (PA14)
- new net SWDIO2: J4.2 (Pin_2), U5.21 (PA13)
- new net SWDIO3: J5.2 (Pin_2), J6.2 (Pin_2), U7.21 (PA13)
- new net SWDIO4: U9.21 (PA13)
- no-connect marks 11 -> 44
Other:
- note added: "ESC1"
- note added: "ESC2"
- note added: "ESC3"
- moved on the sheet: +10ppm1, C1, C10, C11, C12, C13, C14, C15, C16, C17, C18, C19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

Commit message: Update Dragonfly.kicad_sch
Connections:
- net PA10 is gone; now on net PWM3: U1.43 (PA10)
- net PA11 is gone; now on net PWM4: U1.44 (PA11)
- net PA8 is gone; now on net PWM1: U1.41 (PA8)
- net PA9 is gone; now on net PWM2: U1.42 (PA9)
- net ESC2 C2: no longer C55.2, Q21.2 (D), Q22.3 (S), U10.12 (VS3)
- net ESC2_A2: no longer C54.2, Q19.2 (D), Q20.3 (S), U10.18 (VS1)
- net ESC2_A4: now also C54.2, Q19.2 (D), Q20.3 (S), U10.18 (VS1)
- net ESC2_B2: no longer C56.2, Q23.2 (D), Q24.3 (S), U10.15 (VS2)
- net ESC2_B4: now also C56.2, Q23.2 (D), Q24.3 (S), U10.15 (VS2)
- net ESC2_H012: no longer R81.2, U10.19 (HO1)
- net ESC2_H022: no longer R85.2, U10.16 (HO2)
- net ESC2_H032: no longer R83.2, U10.13 (HO3)
- net ESC2_L012: no longer U10.11 (LO1)
- net ESC2_L022: no longer U10.10 (LO2)
- net ESC2_L032: no longer R79.1, U10.9 (LO3)
- net ESC2_l012: no longer R78.2
- net ESC2_l022: no longer R80.2
- net GND: now also U10.25 (EXP), U4.25 (EXP), U6.25 (EXP), U8.25 (EXP)
- new net ESC2 C4: C55.2, Q21.2 (D), Q22.3 (S), U10.12 (VS3)
- new net ESC2_H014: R81.2, U10.19 (HO1)
- new net ESC2_H024: R85.2, U10.16 (HO2)
- new net ESC2_H034: R83.2, U10.13 (HO3)
- new net ESC2_L014: U10.11 (LO1)
- new net ESC2_L024: U10.10 (LO2)
- new net ESC2_L034: R79.1, U10.9 (LO3)
- new net ESC2_l014: R78.2
- new net ESC2_l024: R80.2
Other:
- note added: "ESC4"
