File: PCB/Dragonfly/Dragonfly.kicad_sch (KiCad schematic)
At the start: 201 parts, among them J1 Conn_01x04_Pin, J2 Micro_SD_Card, J3 Conn_01x02_Pin, J4 Conn_01x02_Pin, J5 Conn_01x02_Pin, J6 Conn_01x02_Pin, Q1 Q_NMOS_GDS, Q10 Q_NMOS_GDS, Q11 Q_NMOS_GDS, Q12 Q_NMOS_GDS, Q13 Q_NMOS_GDS, Q14 Q_NMOS_GDS, Q15 Q_NMOS_GDS, Q16 Q_NMOS_GDS, Q17 Q_NMOS_GDS, Q18 Q_NMOS_GDS, Q19 Q_NMOS_GDS, Q2 Q_NMOS_GDS, Q20 Q_NMOS_GDS, Q21 Q_NMOS_GDS, Q22 Q_NMOS_GDS, Q23 Q_NMOS_GDS, Q24 Q_NMOS_GDS, Q3 Q_NMOS_GDS, Q4 Q_NMOS_GDS, Q5 Q_NMOS_GDS, Q6 Q_NMOS_GDS, Q7 Q_NMOS_GDS, Q8 Q_NMOS_GDS, Q9 Q_NMOS_GDS, SW1 SW_SPST, SW2 SW_SPST, U1 STM32F405RGTx, U10 FD6288Q, U2 ICM-20602, U3 AT32F421G8U7, U4 FD6288Q, U5 AT32F421G8U7, U6 FD6288Q, U7 AT32F421G8U7, U8 FD6288Q, U9 AT32F421G8U7, X1 TSX-3225

Commit message: updates
Parts:
- removed D1: blue, symbol Device:D
- removed D2: red, symbol Device:D
- added C57, C60, C62: 10uf, symbol Device:C
- added C58: 0.01uf, symbol Device:C
- added C59: 220uf, symbol Device:C_US
- added C61, C63: 1uf, symbol Device:C
- added C64, C65: 100nf, symbol Device:C
- added D1: LED BLUE, symbol Device:LED
- added D15: 40V, 3A Schottky, Diode_SMD:D_SMC, symbol Diode:B340
- added D16: 40V, 3A Schottky, symbol Device:D_Schottky
- added D2: LED RED, symbol Device:LED
- added J7: Conn_01x02, symbol Connector_Generic:Conn_01x02
- added L2: 15uh, symbol Device:L_Ferrite
- added R87: 30.9k, symbol Device:R
- added R88: 10k, symbol Device:R
- added R89: 100k, symbol Device:R
- added U11: TPS5430DDA, Package_SO:TI_SO-PowerPAD-8_ThermalVias, symbol Regulator_Switching:TPS5430DDA
- added U12: AMS1117-3.3, Package_TO_SOT_SMD:SOT-223-3_TabPin2, symbol Regulator_Linear:AMS1117-3.3
- added U13: L78L08_SO8, Package_SO:SOIC-8_3.9x4.9mm_P1.27mm, symbol Regulator_Linear:L78L08_SO8
Connections:
- net +8V: now also C65.1, U13.1 (OUT)
- net GND: now also C57.2, C59.2, C64.2, C65.2, D1.2 (A), D15.2 (A), D2.2 (A), J7.2 (Pin_2), R88.2, U11.6 (GND), U11.9 (GNDPAD), U13.2 (GND), U13.3 (GND), U13.6 (GND), U13.7 (GND)
- net VDD33: now also C60.1, C61.1, U12.2 (VO)
- net VIN: now also C57.1, C64.1, D16.2 (A), R89.1, U11.7 (VIN), U13.8 (IN)
- net at R4.2: now also D1.1 (K)
- net at R5.2: now also D2.1 (K)
- new net: C60.2, C61.2, C62.2, C63.2
- new net: R89.2, U11.5 (EN)
- new net: R87.2, R88.1, U11.4 (VSENSE)
- new net: C58.1, U11.1 (BOOT)
- new net: C58.2, D15.1 (K), L2.1, U11.8 (PH)
- new net: D16.1 (K), J7.1 (Pin_1)
- new net VOUT: C59.1, C62.1, C63.1, L2.2, R87.1, U12.3 (VI)
Other:
- note added: "Battery connection"
- note added: "Power - Buck (5V) + LDO (3.3V)"
- moved on the sheet: +10ppm1, C1, C10, C11, C12, C13, C14, C15, C16, C17, C18, C19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

Commit message: Update Dragonfly.kicad_sch
Parts:
- added C66, C67, C68, C69: 100nf, symbol Device:C
- added C70, C71: 47uf, symbol Device:C_Polarized
- added J10: USB_C_Receptacle_USB2.0_16P, symbol Connector:USB_C_Receptacle_USB2.0_16P
- added J8: VIN, symbol Connector:Conn_01x02_Socket
- added J9: VOUT, symbol Connector:Conn_01x02_Socket
- added R90, R91: 75 Ω, symbol Device:R
- added R92, R93: 22k, symbol Device:R
- added U14: AT7456E, SOP65P637X110-28N, symbol MAX7456EUI:MAX7456EUI+
- added Y1: 27MHZ, symbol Device:Crystal
Connections:
- net GND: now also C66.2, C67.2, C68.2, J10.A1 (GND), J10.A12 (GND), J10.B1 (GND), J10.B12 (GND), J10.SH (SHIELD), J8.2 (Pin_2), J9.2 (Pin_2), R90.2, U14.20 (AGND), U14.23 (PGND), U14.4 (DGND)
- net VIN: now also C69.1, U14.22 (VIN)
- net VOUT: now also C70.1, U14.26 (VOUT)
- net CS 1 renamed CS IMU
- net MISO renamed MISO IMU
- net MOSI renamed MOSI IMU
- net PB12 renamed CS SOD
- net CS SOD: now also U14.8 (~{CS})
- net PB13 renamed SCK SOD
- net SCK SOD: now also U14.10 (SCLK)
- net PB14 renamed MISO SOD
- net MISO SOD: now also U14.9 (SDIN)
- net PB15 renamed MOSI OSD
- net MOSI OSD: now also U14.11 (SDOUT)
- net SCK renamed SCK IMU
- new net: J9.1 (Pin_1), R91.1
- new net: C70.2, C71.2, R91.2
- new net: J10.A5 (CC1), R92.1
- new net: C69.2, J8.1 (Pin_1), R90.1
- new net: J10.B5 (CC2), R93.1
- new net +5V: J10.A4 (VBUS), J10.A9 (VBUS), J10.B4 (VBUS), J10.B9 (VBUS), R92.2, R93.2
- new net 5V: C66.1, C67.1, C68.1, U14.19 (~{RESET}), U14.21 (AVDD), U14.24 (PVDD), U14.3 (DVDD)
- new net D+: J10.A6 (D+), J10.B6 (D+)
- new net D-: J10.A7 (D-), J10.B7 (D-)
- new net SAG: C71.1, U14.25 (SAG)
- new net XTAL1: U14.5 (CLKIN), Y1.1
- new net XTAL2: U14.6 (XFB), Y1.2
- no-connect marks 44 -> 49
Other:
- note added: "OSD - AT7456E"
- note added: "USB-C 16pin"
- moved on the sheet: C20, C5, C57, C58, C59, C60, C61, C62, C63, C64, C65, D15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

Commit message: Update Dragonfly.kicad_sch
Parts:
- removed J10: USB_C_Receptacle_USB2.0_16P, symbol Connector:USB_C_Receptacle_USB2.0_16P
- removed R92, R93: 22k, symbol Device:R
- added C72: 1uf, symbol Device:C
- added C73: 0.1uf, symbol Device:C
- added U15: BMP280, Package_LGA:Bosch_LGA-8_2x2.5mm_P0.65mm_ClockwisePinNumbering, symbol Sensor_Pressure:BMP280
- J8: value VIN -> CAM VIN
Connections:
- net ESC2 C1 is gone; now on net ESC2_C1: C24.2, Q1.2 (D), Q2.3 (S), U4.12 (VS3)
- net ESC2 C2 is gone; now on net ESC2_C2: C37.2, Q10.3 (S), Q9.2 (D), U6.12 (VS3)
- net ESC2 C3 is gone; now on net ESC2_C3: C46.2, Q15.2 (D), Q16.3 (S), U8.12 (VS3)
- net ESC2 C4 is gone; now on net ESC2_C4: C55.2, Q21.2 (D), Q22.3 (S), U10.12 (VS3)
- net ESC2_l011 is gone; now on net ESC2_L011: R24.2
- net ESC2_l012 is gone; now on net ESC2_L012: R38.2
- net ESC2_l013 is gone; now on net ESC2_L013: R58.2
- net ESC2_l014 is gone; now on net ESC2_L014: R78.2
- net ESC2_l021 is gone; now on net ESC2_L021: R21.2
- net ESC2_l022 is gone; now on net ESC2_L022: R40.2
- net ESC2_l023 is gone; now on net ESC2_L023: R60.2
- net ESC2_l024 is gone; now on net ESC2_L024: R80.2
- net VDD33A is gone; now on net VDD33: C13.1, C14.1, L1.2, U1.13 (VDDA)
- net 5V: now also C62.1, C63.1, U12.3 (VI)
- net GND: now also C60.2, C61.2, C62.2, C63.2, U12.1 (GND), U2.10 (RESV), U2.11 (RESV), U2.12 (RESV), U2.13 (GND), U2.15 (RESV), U2.8 (FSYNC), U2.9 (RESV), C72.2, C73.2, U15.1 (GND), U15.7 (GND)
- net HI12: no longer U10.22 (HIN1)
- net HI14: now also U10.22 (HIN1)
- net HI22: no longer U10.23 (HIN2)
- net HI24: now also U10.23 (HIN2)
- net HI32: no longer U10.24 (HIN3)
- net HI34: now also U10.24 (HIN3)
- net LI12: no longer U10.1 (LIN1)
- net LI14: now also U10.1 (LIN1)
- net LI22: no longer U10.2 (LIN2)
- net LI24: now also U10.2 (LIN2)
- net LI32: no longer U10.3 (LIN3)
- net LI34: now also U10.3 (LIN3)
- net MISO SOD: now also U14.11 (SDOUT); no longer U14.9 (SDIN)
- net MOSI OSD: now also U14.9 (SDIN); no longer U14.11 (SDOUT)
- net SWCLK3: no longer J6.1 (Pin_1)
- net SWCLK4: now also J6.1 (Pin_1)
- net SWDIO3: no longer J6.2 (Pin_2)
- net SWDIO4: now also J6.2 (Pin_2)
- net VDD33: now also C72.1, C73.1, U15.6 (VDDIO), U15.8 (VDD)
- net VOUT: no longer C62.1, C63.1, U12.3 (VI)
- net PA13 renamed SWDIO
- net PA14 renamed SWCLK
- net PB5 renamed SCK B
- net SCK B: now also U15.4 (SCK)
- net PB6 renamed MOSI B
- net MOSI B: now also U15.3 (SDI)
- net PB7 renamed MISO B
- net MISO B: now also U15.5 (SDO)
- net PB8 renamed CSB
- net CSB: now also U15.2 (CSB)
- no-connect marks 49 -> 67
Other:
- note added: "BMP280 Barometer"
- note removed: "USB-C 16pin"
- moved on the sheet: +10ppm1, C1, C10, C11, C12, C13, C14, C15, C16, C17, C18, C19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

Commit message: updated
Parts:
- removed D16: 40V, 3A Schottky, symbol Device:D_Schottky
- removed J7: Conn_01x02, symbol Connector_Generic:Conn_01x02
- added J7: XT60PW-M, XT60PW-M:AMASS_XT60PW-M, symbol XT60PW-M:XT60PW-M
- +10ppm1, Y1: footprint (none) -> Crystal:Crystal_SMD_3225-4Pin_3.2x2.5mm
- C1, C10, C11, C12, C13, C14, C15, C17, C18, C19, C2, C20, C21, C22, C23, C24, C25, C26, C27, C28, C29, C3, C30, C31, C32, C33, C34, C35, C36, C37, C38, C39, C4, C40, C41, C42, C43, C44, C45, C46, C47, C48, C49, C5, C50, C51, C52, C53, C54, C55, C56, C57, C58, C6, C60, C61, C62, C63, C64, C65, C66, C67, C68, C69, C70, C71, C72, C73, C9: footprint (none) -> Capacitor_SMD:C_0402_1005Metric
- C16: value 4.7uF -> 4.7uf; footprint (none) -> Capacitor_SMD:C_0402_1005Metric
- C59: footprint (none) -> Capacitor_SMD:CP_Elec_6.3x5.8
- C7, C8: value 2.2uF -> 2.2uf; footprint (none) -> Capacitor_SMD:C_0402_1005Metric
- D1, D2: footprint (none) -> LED_SMD:LED_0201_0603Metric
- J1: footprint (none) -> Connector_JST:JST_EH_B4B-EH-A_1x04_P2.50mm_Vertical
- J2: footprint (none) -> Connector_Card:microSD_HC_Molex_104031-0811
- J3, J4, J5, J6, J8, J9: footprint (none) -> Connector_JST:JST_EH_S2B-EH_1x02_P2.50mm_Horizontal
- L1: footprint (none) -> Inductor_SMD:L_0402_1005Metric
- L2: footprint (none) -> Inductor_SMD_Wurth:L_Wurth_WE-LQSH-4020
- R1, R10, R11, R12, R13, R14, R15, R16, R17, R18, R19, R2, R20, R21, R22, R23, R24, R25, R26, R27, R28, R29, R3, R30, R31, R32, R33, R34, R35, R36, R37, R38, R39, R4, R40, R41, R42, R43, R44, R45, R46, R47, R48, R49, R5, R50, R51, R52, R53, R54, R55, R56, R57, R58, R59, R6, R60, R61, R62, R63, R64, R65, R66, R67, R68, R69, R7, R70, R71, R72, R73, R74, R75, R76, R77, R78, R79, R8, R80, R81, R82, R83, R84, R85, R86, R88, R89, R9: footprint (none) -> Resistor_SMD:R_0402_1005Metric
- R87: footprint (none) -> Resistor_SMD:R_0815_2038Metric
- R90, R91: value 75 Ω -> 75R; footprint (none) -> Resistor_SMD:R_0402_1005Metric
- SW1, SW2: footprint (none) -> Button_Switch_SMD:SW_SPST_EVQP7A
- U10, U4, U6, U8: footprint QFN50P400X400X90-25N -> FD6288Q:QFN50P400X400X90-25N
- U14: footprint SOP65P637X110-28N -> AT7456E:SOP65P640X120-29N
- U3, U5, U7, U9: footprint AT32F421G8U7:AT32F421G8U7 -> Library:AT32F421G8U7
- X1: footprint TSX-3225 -> TSX-3225:TSX-3225
Connections:
- net GND: now also J7.2 (N), J7.SH1 (SHIELD), J7.SH2 (SHIELD)
- net VIN: now also J7.1 (P)
Other:
- moved on the sheet: J1

Commit message: Update Dragonfly.kicad_sch
Parts:
- J3, J4, J5, J6, J8, J9: footprint Connector_JST:JST_EH_S2B-EH_1x02_P2.50mm_Horizontal -> Connector_JST:JST_EH_B2B-EH-A_1x02_P2.50mm_Vertical
- Q1, Q10, Q11, Q12, Q13, Q14, Q15, Q16, Q17, Q18, Q19, Q2, Q20, Q21, Q22, Q23, Q24, Q3, Q4, Q5, Q6, Q7, Q8, Q9: footprint (none) -> Package_SON:Diodes_PowerDI3333-8
- SW1, SW2: footprint Button_Switch_SMD:SW_SPST_EVQP7A -> Button_Switch_SMD:SW_Tactile_SPST_NO_Straight_CK_PTS636Sx25SMTRLFS
- U3, U5, U7, U9: footprint Library:AT32F421G8U7 -> AT7456E:SOP65P640X120-29N
Connections:
- net VDD33: no longer C14.1, L1.2
- new net: C14.1, L1.2
Other:
- moved on the sheet: C72, C73, U15

Commit message: update
Parts:
- removed C15: 100nf, Capacitor_SMD:C_0402_1005Metric, symbol Device:C
- removed C16: 4.7uf, Capacitor_SMD:C_0402_1005Metric, symbol Device:C
- removed J2: Micro_SD_Card, Connector_Card:microSD_HC_Molex_104031-0811, symbol Connector:Micro_SD_Card
- removed R6: 0R, Resistor_SMD:R_0402_1005Metric, symbol Device:R
- U3, U5, U7, U9: footprint AT7456E:SOP65P640X120-29N -> Library:AT32F421G8U7
Connections:
- no-connect marks 67 -> 73
Other:
- note removed: "TF interface"
