File: PCB/Dragonfly/Dragonfly.kicad_pcb (KiCad board)
At the start: 2 copper layers, 66 x 58.8 mm, 230 parts, among them J1 Conn_01x04_Pin, J3 Conn_01x02_Pin, J4 Conn_01x02_Pin, J5 Conn_01x02_Pin, J6 Conn_01x02_Pin, J7 XT60PW-M, J8 CAM VIN, J9 VOUT, Q1 Q_NMOS_GDS, Q10 Q_NMOS_GDS, Q11 Q_NMOS_GDS, Q12 Q_NMOS_GDS, Q13 Q_NMOS_GDS, Q14 Q_NMOS_GDS, Q15 Q_NMOS_GDS, Q16 Q_NMOS_GDS, Q17 Q_NMOS_GDS, Q18 Q_NMOS_GDS, Q19 Q_NMOS_GDS, Q2 Q_NMOS_GDS, Q20 Q_NMOS_GDS, Q21 Q_NMOS_GDS, Q22 Q_NMOS_GDS, Q23 Q_NMOS_GDS, Q24 Q_NMOS_GDS, Q3 Q_NMOS_GDS, Q4 Q_NMOS_GDS, Q5 Q_NMOS_GDS, Q6 Q_NMOS_GDS, Q7 Q_NMOS_GDS, Q8 Q_NMOS_GDS, Q9 Q_NMOS_GDS, SW1 SW_SPST, SW2 SW_SPST, U1 STM32F405RGTx, U10 FD6288Q, U11 TPS5430DDA, U12 AMS1117-3.3, U13 L78L08_SO8, U14 AT7456E, U15 BMP280, U2 ICM-20602, U3 AT32F421G8U7, U4 FD6288Q, U5 AT32F421G8U7, U6 FD6288Q, U7 AT32F421G8U7, U8 FD6288Q, U9 AT32F421G8U7, X1 TSX-3225, Y1 27MHZ

Commit message: Update Dragonfly.kicad_pcb
Parts:
- removed J3, J4, J5, J6: Conn_01x02_Pin, Connector_JST:JST_EH_B2B-EH-A_1x02_P2.50mm_Vertical
- added TP10: VDD33, TestPoint:TestPoint_Pad_D1.0mm, B.Cu at (281.9, 104.0)
- added TP11: GND, TestPoint:TestPoint_Pad_D1.0mm, B.Cu at (277.8, 104.1)
- added TP12: SWCLK3, TestPoint:TestPoint_Pad_D1.0mm, B.Cu at (282.0, 100.7)
- added TP13: SWDIO3, TestPoint:TestPoint_Pad_D1.0mm, B.Cu at (277.9, 100.8)
- added TP14: VDD33, TestPoint:TestPoint_Pad_D1.0mm, B.Cu at (257.6, 104.4)
- added TP15: GND, TestPoint:TestPoint_Pad_D1.0mm, B.Cu at (254.7, 104.4)
- added TP16: SWCLK4, TestPoint:TestPoint_Pad_D1.0mm, B.Cu at (257.7, 101.0)
- added TP17: SWDIO4, TestPoint:TestPoint_Pad_D1.0mm, B.Cu at (254.9, 101.1)
- added TP2: VDD33, TestPoint:TestPoint_Pad_D1.0mm, B.Cu at (281.8, 112.4)
- added TP3: GND, TestPoint:TestPoint_Pad_D1.0mm, B.Cu at (277.7, 112.4)
- added TP4: SWCLK1, TestPoint:TestPoint_Pad_D1.0mm, B.Cu at (281.9, 115.8)
- added TP5: SWDIO1, TestPoint:TestPoint_Pad_D1.0mm, B.Cu at (277.8, 115.8)
- added TP6: VDD33, TestPoint:TestPoint_Pad_D1.0mm, B.Cu at (257.9, 111.8)
- added TP7: GND, TestPoint:TestPoint_Pad_D1.0mm, B.Cu at (255.0, 111.8)
- added TP8: SWCLK2, TestPoint:TestPoint_Pad_D1.0mm, B.Cu at (258.0, 115.2)
- added TP9: SWDIO2, TestPoint:TestPoint_Pad_D1.0mm, B.Cu at (255.3, 115.2)
- C28, C31, C32, C33, C34, C35, C36, C37, C38, C39, C40, C41, C42, C43, C44, C45, C46, C47, C48, C49, C50, C51, C52, C53, C54, C55, C56, D10, D11, D12, D13, D14, D6, D7, D8, D9, Q10, Q11, Q12, Q13, Q14, Q15, Q16, Q17, Q18, Q19, Q20, Q21, Q22, Q23, Q24, Q7, Q8, Q9, R27, R28, R29, R30, R31, R32, R33, R34, R35, R36, R37, R38, R39, R40, R41, R42, R43, R44, R45, R46, R47, R48, R49, R50, R51, R52, R53, R54, R55, R56, R57, R58, R59, R60, R61, R62, R63, R64, R65, R66, R67, R68, R69, R70, R71, R72, R73, R74, R75, R76, R77, R78, R79, R80, R81, R82, R83, R84, R85, R86, U10, U5, U6, U7, U8, U9: moved to B.Cu
- moved R51 171.0 mm to (295.9, 93.9), turned to 90 degrees
- moved R47 170.2 mm to (295.9, 91.9), turned to -90 degrees
- moved R53 166.3 mm to (295.9, 89.9), turned to -90 degrees
- moved R64 165.3 mm to (291.4, 85.4), turned to 180 degrees
- moved R59 163.0 mm to (291.3, 87.6), turned to 180 degrees
- moved R63 161.7 mm to (288.5, 87.1), turned to -90 degrees
- moved R57 161.5 mm to (291.4, 103.8)
- moved R60 161.0 mm to (288.4, 84.7), turned to -90 degrees
- moved R50 160.6 mm to (287.1, 105.8), turned to 180 degrees
- moved R61 160.6 mm to (289.3, 95.9), turned to -90 degrees
- moved R48 160.5 mm to (287.0, 102.5)
- moved R49 160.5 mm to (287.0, 104.7)
- moved R56 159.6 mm to (289.4, 103.7), turned to 180 degrees
- moved R62 159.5 mm to (287.9, 95.4), turned to -90 degrees
- moved Q13 157.8 mm to (282.6, 96.6)
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
Commit message: updated
Parts:
- added REF**: MountingHole_2.1mm, MountingHole:MountingHole_2.1mm, F.Cu at (238.0, 135.0)
- added REF**: MountingHole_2.1mm, MountingHole:MountingHole_2.1mm, F.Cu at (297.9, 135.5)
- added REF**: MountingHole_2.1mm, MountingHole:MountingHole_2.1mm, F.Cu at (298.4, 82.5)
- added REF**: MountingHole_2.1mm, MountingHole:MountingHole_2.1mm, F.Cu at (238.5, 82.3)
- C7, C72, C73, C8: moved to B.Cu
- R18, R22, R26, R42, R44, R46, R62, R64, R66, R82, R84, R86: value 10k -> 0R
- moved J7 104.0 mm to (268.1, 129.9)
- moved C12 99.8 mm to (247.3, 107.8)
- moved C14 99.8 mm to (247.3, 105.5)
- moved C13 99.8 mm to (247.3, 104.3)
- moved C2 99.8 mm to (247.3, 109.0)
- moved C6 99.8 mm to (247.3, 110.2)
- moved C9 99.8 mm to (247.3, 106.6)
- moved C5 99.7 mm to (257.8, 119.0)
- moved R1 99.7 mm to (249.8, 119.0)
- moved SW1 99.7 mm to (253.8, 116.9)
- moved R3 99.6 mm to (258.4, 122.9)
- moved R2 99.6 mm to (249.6, 122.8)
- moved SW2 99.6 mm to (253.9, 121.3)
- moved Y1 99.1 mm to (275.3, 94.1)
- moved R90 98.8 mm to (278.9, 92.3)
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Routing:
- net GND: track 0.00 -> 136.7 mm, vias 0 -> 108
- net VDD33: track 0.00 -> 53.4 mm, vias 0 -> 26
- added copper zone on In2.Cu, net GND
- added copper zone on In1.Cu, net VDD33
Other:
- copper layers 2 -> 4

Commit message: Update Dragonfly.kicad_pcb
Parts:
- removed REF** (x4): MountingHole_2.1mm, MountingHole:MountingHole_2.1mm
- moved R91 18.4 mm to (291.7, 108.5), turned to 90 degrees
- moved R7 1.04 mm to (289.5, 111.7)
- moved R8 1.04 mm to (291.4, 111.7)
- moved TP5 0.75 mm to (278.5, 115.8)
- moved TP3 0.66 mm to (278.4, 112.4)
- moved TP4 0.58 mm to (281.4, 116.0)
- moved C23 0.48 mm to (288.0, 123.6)
- moved TP11 0.41 mm to (278.2, 104.1)
- moved TP12 0.29 mm to (281.9, 101.0)
- moved TP13 0.28 mm to (278.0, 101.0)
- moved C22 0.19 mm to (292.4, 120.0)
- moved C21 0.19 mm to (291.4, 120.0)
- moved C27 0.10 mm to (295.7, 120.1)
Connections:
- C18 pad 1: VDD -> VDD33
- C19 pad 1: VDD -> VDD33
- C20 pad 1: VDD -> VDD33
- U2 pad 1: VDD -> VDD33
- U2 pad 16: VDD -> VDD33
Routing:
- net VIN: track 0.00 -> 243.6 mm, vias 0 -> 12
- net +8V: track 0.00 -> 71.2 mm, vias 0 -> 7
- net BOOT0: track 0.00 -> 45.6 mm, vias 0 -> 1
- net ESC2_B1: track 0.00 -> 37.7 mm, vias 0 -> 5
- net PWM4: track 0.00 -> 37.2 mm, vias 0 -> 1
- net Net-(C70-Pad2): track 0.00 -> 34.2 mm, vias 0 -> 2
- net Net-(D15-K): track 0.00 -> 33.3 mm
- net 5V: track 0.00 -> 33.1 mm
- net ESC2_C3: track 0.00 -> 32.6 mm, vias 0 -> 2
- net Net-(U3-PA1): track 0.00 -> 30.8 mm, vias 0 -> 4
- net ESC2_A1: track 0.01 -> 30.3 mm
- net PWM2: track 0.00 -> 30.3 mm, vias 0 -> 1
- net PWM1: track 0.00 -> 26.8 mm, vias 0 -> 1
- net ESC2_C1: track 0.00 -> 26.0 mm, vias 0 -> 4
- net CS SOD: track 0.00 -> 23.4 mm, vias 0 -> 2
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
Commit message: Update Dragonfly.kicad_pcb
Parts:
- moved C59 33.1 mm to (280.5, 87.7), turned to 180 degrees
- moved C66 21.8 mm to (271.6, 93.0)
- moved C67 21.4 mm to (271.6, 92.0)
- moved C68 21.1 mm to (271.6, 90.7)
- moved C70 20.9 mm to (271.3, 88.9), turned to 90 degrees
- moved L2 19.7 mm to (264.6, 90.8)
- moved C71 19.3 mm to (272.5, 88.9), turned to 90 degrees
- moved C69 19.1 mm to (273.9, 88.9), turned to 90 degrees
- moved C44 14.5 mm to (274.6, 96.9), turned to 0 degrees
- moved R70 14.1 mm to (262.5, 100.7), turned to -90 degrees
- moved R69 12.5 mm to (261.2, 100.7), turned to -90 degrees
- moved R78 10.0 mm to (242.9, 88.7), turned to 0 degrees
- moved C52 9.62 mm to (242.4, 87.0)
- moved C50 9.62 mm to (243.4, 87.0)
- moved R87 9.53 mm to (259.2, 101.0), turned to 90 degrees
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Routing:
- net +8V: track 71.2 -> 190.9 mm, vias 7 -> 26
- net ESC2_B3: track 0.00 -> 59.3 mm, vias 0 -> 12
- net ESC2_B2: track 0.00 -> 48.7 mm, vias 0 -> 12
- net VOUT: track 6.47 -> 50.8 mm, vias 0 -> 9
- net Net-(J8-Pin_1): track 11.0 -> 51.5 mm, vias 0 -> 5
- net ESC2_A2: track 0.00 -> 40.0 mm, vias 0 -> 2
- net ESC2_A3: track 0.00 -> 39.9 mm, vias 0 -> 5
- net BOOT0: track 45.6 -> 82.1 mm, vias 1 -> 3
- net Net-(U9-PA1): track 0.00 -> 36.1 mm, vias 0 -> 11
- net ESC2_C4: track 0.00 -> 33.4 mm, vias 0 -> 2
- net Net-(U5-PA1): track 0.00 -> 32.4 mm, vias 0 -> 4
- net ESC2_B4: track 0.00 -> 29.8 mm, vias 0 -> 7
- net SWDIO3: track 0.00 -> 28.6 mm, vias 0 -> 2
- net Net-(Q14-G): track 0.00 -> 28.2 mm, vias 0 -> 6
- net ESC2_C2: track 0.00 -> 27.7 mm, vias 0 -> 4
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
Commit message: updates
Parts:
- added REF**: MountingHole_2.2mm_M2_DIN965_Pad_TopBottom, MountingHole:MountingHole_2.2mm_M2_DIN965_Pad_TopBottom, F.Cu at (238.5, 82.3)
- added REF**: MountingHole_2.2mm_M2_DIN965_Pad_TopBottom, MountingHole:MountingHole_2.2mm_M2_DIN965_Pad_TopBottom, F.Cu at (238.1, 134.9)
- added REF**: MountingHole_2.2mm_M2_DIN965_Pad_TopBottom, MountingHole:MountingHole_2.2mm_M2_DIN965_Pad_TopBottom, F.Cu at (298.2, 82.6)
- added REF**: MountingHole_2.2mm_M2_DIN965_Pad_TopBottom, MountingHole:MountingHole_2.2mm_M2_DIN965_Pad_TopBottom, F.Cu at (297.8, 135.3)
- moved C21 8.96 mm to (294.0, 128.6)
- moved C22 8.96 mm to (295.0, 128.6)
Connections:
- C18 pad 1: VDD33 -> VDD
- C19 pad 1: VDD33 -> VDD
- C20 pad 1: VDD33 -> VDD
- U2 pad 1: VDD33 -> VDD
- U2 pad 16: VDD33 -> VDD
Routing:
- net VDD: track 0.00 -> 9.60 mm, vias 0 -> 2
- net VDD33: track 67.6 -> 62.8 mm, vias 38 -> 35
- net VIN: track 257.2 -> 254.8 mm
- net ESC2_L014: track 5.03 -> 3.42 mm, vias 3 -> 2
- net GND: track 133.2 -> 134.7 mm
- net 5V: track 52.6 -> 51.4 mm, vias 12 -> 11
- net HI31: track 5.91 -> 4.98 mm
- net ESC2_B1: track 37.7 -> 38.5 mm
- net VOUT: track 50.8 -> 50.1 mm
- net ESC2_B3: track 59.3 -> 58.7 mm
- net Net-(U7-BOOT0): track 7.55 -> 6.96 mm
- net ESC2_C3: track 31.4 -> 30.9 mm
- net BOOT0: track 82.1 -> 81.6 mm, vias 3 -> 2
- net ESC2_B4: vias 7 -> 6
- net +8V: track 190.9 -> 191.0 mm, vias 26 -> 25
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