File: PCB/Dragonfly/.history/Dragonfly.kicad_pcb (KiCad board)
At the start: 4 copper layers, 66 x 58.8 mm, 246 parts, among them J1 Conn_01x04_Pin, J7 XT60PW-M, J8 CAM VIN, J9 VOUT, Q1 Q_NMOS_GDS, Q10 Q_NMOS_GDS, Q11 Q_NMOS_GDS, Q12 Q_NMOS_GDS, Q13 Q_NMOS_GDS, Q14 Q_NMOS_GDS, Q15 Q_NMOS_GDS, Q16 Q_NMOS_GDS, Q17 Q_NMOS_GDS, Q18 Q_NMOS_GDS, Q19 Q_NMOS_GDS, Q2 Q_NMOS_GDS, Q20 Q_NMOS_GDS, Q21 Q_NMOS_GDS, Q22 Q_NMOS_GDS, Q23 Q_NMOS_GDS, Q24 Q_NMOS_GDS, Q3 Q_NMOS_GDS, Q4 Q_NMOS_GDS, Q5 Q_NMOS_GDS, Q6 Q_NMOS_GDS, Q7 Q_NMOS_GDS, Q8 Q_NMOS_GDS, Q9 Q_NMOS_GDS, SW1 SW_SPST, SW2 SW_SPST, U1 STM32F405RGTx, U10 FD6288Q, U11 TPS5430DDA, U12 AMS1117-3.3, U13 L78L08_SO8, U14 AT7456E, U15 BMP280, U2 ICM-20602, U3 AT32F421G8U7, U4 FD6288Q, U5 AT32F421G8U7, U6 FD6288Q, U7 AT32F421G8U7, U8 FD6288Q, U9 AT32F421G8U7, X1 TSX-3225, Y1 27MHZ

Commit message: Update Dragonfly.kicad_pcb
Routing:
- net GND: track 132.1 -> 137.3 mm, vias 99 -> 106
Changed lines of the file:
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@@
+	)
+	(segment
+		(start 279.43 92.73)
+		(end 279.6 92.9)
+		(width 0.2)
+		(layer "F.Cu")
+		(net "GND")
 	)
 	(segment
@@
 	)
 	(segment
+		(start 279.43 92.31)
+		(end 279.43 92.73)
+		(width 0.2)
+		(layer "F.Cu")
+		(net "GND")
+	)
+	(segment
 		(start 280.19 111.85)
 		(end 281.9 111.85)
@@
 	(via
 		(at 286.073002 99.9)
+		(size 0.4)
+		(drill 0.2)
+		(layers "F.Cu" "B.Cu")
+		(net "GND")
+	)
+	(via
+		(at 287.236 95.83)
 		(size 0.4)
 		(drill 0.2)
@@
 	)
 	(via
+		(at 279.6 92.9)
+		(size 0.4)
+		(drill 0.2)
+		(layers "F.Cu" "B.Cu")
+		(net "GND")
+	)
+	(via
 		(at 287.36 120.58)
 		(size 0.4)
@@
 	(via
 		(at 248.756505 95.414423)
+		(size 0.4)
+		(drill 0.2)
+		(layers "F.Cu" "B.Cu")
+		(net "GND")
+	)
+	(via
+		(at 276.2 84.3)
 		(size 0.4)
 		(drill 0.2)
@@
 	)
 	(via
+		(at 281.36 94.53)
+		(size 0.4)
+		(drill 0.2)
+		(layers "F.Cu" "B.Cu")
+		(net "GND")
+	)
+	(via
 		(at 248.3 100)
 		(size 0.4)
@@
 	)
 	(via
+		(at 280.1 88.8)
+		(size 0.4)
+		(drill 0.2)
+		(layers "F.Cu" "B.Cu")
+		(net "GND")
+	)
+	(via
 		(at 249.9 106.3)
 		(size 0.4)
@@
 	(via
 		(at 287.265 106.3925)
+		(size 0.4)
+		(drill 0.2)
+		(layers "F.Cu" "B.Cu")
+		(net "GND")
+	)
+	(via
+		(at 276.3 89.7)
 		(size 0.4)
 		(drill 0.2)
@@
 	)
 	(via
+		(at 286.073002 94.5)
+		(size 0.4)
+		(drill 0.2)
+		(layers "F.Cu" "B.Cu")
+		(net "GND")
+	)
+	(via
 		(at 290.72 84.83)
 		(size 0.6)
@@
 	)
 	(segment
+		(start 279.87 88.57)
+		(end 280.1 88.8)
+		(width 0.2)
+		(layer "B.Cu")
+		(net "GND")
+	)
+	(segment
 		(start 277.707142 112.37)
 		(end 279.36 112.37)
@@
 	)
 	(segment
+		(start 279.41 88.57)
+		(end 279.87 88.57)
+		(width 0.2)
+		(layer "B.Cu")
+		(net "GND")
+	)
+	(segment
 		(start 245.36 128.76)
 		(end 245.4 128.8)
@@
 	)
 	(segment
+		(start 276.45 89.85)
+		(end 276.3 89.7)
+		(width 0.2)
+		(layer "B.Cu")
+		(net "GND")
+	)
+	(segment
 		(start 240.76 123.01)
 		(end 241.39 123.01)
@@
 	)
 	(segment
+		(start 281.1 94.79)
+		(end 281.36 94.53)
+		(width 0.2)
+		(layer "B.Cu")
+		(net "GND")
+	)
+	(segment
 		(start 252.25 95.05)
 		(end 252.2 95)
@@
 	)
 	(segment
+		(start 285.99 95.05)
+		(end 285.99 94.583002)
+		(width 0.2)
+		(layer "B.Cu")
+		(net "GND")
+	)
+	(segment
 		(start 290.85 84.96)
 		(end 290.72 84.83)
@@
 	)
 	(segment
+		(start 276.22 84.32)
+		(end 276.2 84.3)
+		(width 0.2)
+		(layer "B.Cu")
+		(net "GND")
+	)
+	(segment
 		(start 241.13 101.082282)
 		(end 241.13 99.172282)
@@
 	)
 	(segment
+		(start 276.22 84.89)
+		(end 276.22 84.32)
+		(width 0.2)
+		(layer "B.Cu")
+		(net "GND")
+	)
+	(segment
 		(start 247.402282 85.102282)
 		(end 247.2 84.9)
@@
 	)
 	(segment
+		(start 287.92 95.9)
+		(end 287.306 95.9)
+		(width 0.2)
+		(layer "B.Cu")
+		(net "GND")
+	)
+	(segment
 		(start 278.23 127.97)
 		(end 277.8 128.4)
@@
 	)
 	(segment
+		(start 287.306 95.9)
+		(end 287.236 95.83)
+		(width 0.2)
+		(layer "B.Cu")
+		(net "GND")
+	)
+	(segment
 		(start 284.02 120.87)
 		(end 285.02 120.87)
@@
 	)
 	(segment
+		(start 281.1 95.64)
+		(end 281.1 94.79)
+		(width 0.2)
+		(layer "B.Cu")
+		(net "GND")
+	)
+	(segment
 		(start 257.96 88.392282)
 		(end 257.96 87.96)
@@
 	)
 	(segment
+		(start 276.45 90.26)
+		(end 276.45 89.85)
+		(width 0.2)
+		(layer "B.Cu")
+		(net "GND")
+	)
+	(segment
 		(start 245.975 116.695)
 		(end 245.975 117.92)
 		(width 0.2)
 		(layer "B.Cu")
+		(net "GND")
+	)
+	(segment
+		(start 285.99 94.583002)
+		(end 286.073002 94.5)
+		(width 0.2)
+		(layer "B.Cu")

Commit message: updated
Routing:
- net VDD33: track 0.00 -> 52.1 mm, vias 0 -> 25
- net GND: track 137.3 -> 136.7 mm, vias 106 -> 108
- added copper zone on In1.Cu, net VDD33

Commit message: Update Dragonfly.kicad_pcb
Parts:
- removed REF** (x4): MountingHole_2.1mm, MountingHole:MountingHole_2.1mm
- moved R91 18.4 mm to (291.7, 108.5), turned to 90 degrees
- moved R7 1.04 mm to (289.5, 111.7)
- moved R8 1.04 mm to (291.4, 111.7)
- moved TP5 0.75 mm to (278.5, 115.8)
- moved TP3 0.66 mm to (278.4, 112.4)
- moved TP4 0.58 mm to (281.4, 116.0)
- moved C23 0.48 mm to (288.0, 123.6)
- moved TP11 0.41 mm to (278.2, 104.1)
- moved TP12 0.29 mm to (281.9, 101.0)
- moved TP13 0.28 mm to (278.0, 101.0)
- moved C22 0.19 mm to (292.4, 120.0)
- moved C21 0.19 mm to (291.4, 120.0)
- moved C27 0.10 mm to (295.7, 120.1)
Connections:
- C18 pad 1: VDD -> VDD33
- C19 pad 1: VDD -> VDD33
- C20 pad 1: VDD -> VDD33
- U2 pad 1: VDD -> VDD33
- U2 pad 16: VDD -> VDD33
Routing:
- net VIN: track 0.00 -> 229.5 mm, vias 0 -> 11
- net +8V: track 0.00 -> 71.2 mm, vias 0 -> 7
- net BOOT0: track 0.00 -> 45.6 mm, vias 0 -> 1
- net ESC2_B1: track 0.00 -> 37.7 mm, vias 0 -> 5
- net PWM4: track 0.00 -> 37.2 mm, vias 0 -> 1
- net Net-(C70-Pad2): track 0.00 -> 34.2 mm, vias 0 -> 2
- net Net-(D15-K): track 0.00 -> 33.3 mm
- net 5V: track 0.00 -> 33.1 mm
- net Net-(U3-PA1): track 0.00 -> 30.8 mm, vias 0 -> 4
- net ESC2_A1: track 0.01 -> 30.3 mm
- net PWM2: track 0.00 -> 30.3 mm, vias 0 -> 1
- net PWM1: track 0.00 -> 26.8 mm, vias 0 -> 1
- net ESC2_C1: track 0.00 -> 26.0 mm, vias 0 -> 4
- net CS SOD: track 0.00 -> 23.4 mm, vias 0 -> 2
- net SWDIO: track 0.00 -> 23.3 mm
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
Commit message: Update Dragonfly.kicad_pcb
Routing:
- net ESC2_C3: track 0.00 -> 32.6 mm, vias 0 -> 2
- net Net-(Q15-S): track 0.00 -> 19.1 mm
- net VIN: track 229.5 -> 243.6 mm, vias 11 -> 12
- net Net-(Q16-G): track 0.00 -> 9.24 mm, vias 0 -> 2
- net XTAL1: track 0.00 -> 7.91 mm
- net XTAL2: track 0.00 -> 5.28 mm
- net Net-(U7-PA5): track 0.00 -> 4.50 mm
- net Net-(D10-K): track 0.00 -> 2.73 mm
- net ESC2_L033: track 0.00 -> 2.68 mm

Commit message: Update Dragonfly.kicad_pcb
Parts:
- moved C44 14.5 mm to (274.6, 96.9), turned to 0 degrees
- moved C43 3.27 mm to (295.6, 95.7), turned to 0 degrees
- moved C41 2.70 mm to (294.1, 96.2)
- moved R56 1.44 mm to (289.9, 105.1)
- moved R57 1.44 mm to (291.9, 105.1)
- moved TP13 1.01 mm to (278.2, 102.0)
- moved TP12 0.96 mm to (281.9, 102.0)
- moved U8 0.82 mm to (291.8, 91.3)
- moved C70 0.42 mm to (291.6, 94.4), turned to 0 degrees
- moved R50 0.33 mm to (287.0, 106.1)
- moved C45 0.30 mm to (285.9, 97.9)
- moved R49 0.16 mm to (287.0, 104.9)
- moved R55 0.07 mm to (287.0, 103.7)
- turned R65 to 0 degrees
Routing:
- net SWDIO3: track 0.00 -> 28.2 mm, vias 0 -> 2
- net SWCLK3: track 0.00 -> 23.4 mm, vias 0 -> 2
- net +8V: track 71.2 -> 85.3 mm, vias 7 -> 9
- net ESC2_B3: track 0.00 -> 11.8 mm, vias 0 -> 2
- net ESC2_A3: track 0.00 -> 9.43 mm
- net Net-(Q18-G): track 0.00 -> 7.78 mm, vias 0 -> 2
- net Net-(U7-PA0): track 0.00 -> 7.64 mm
- net Net-(U7-BOOT0): track 0.00 -> 7.55 mm
- net Net-(U7-PA1): track 0.00 -> 6.00 mm
- net HI13: track 0.00 -> 5.77 mm
- net GND: track 142.8 -> 137.3 mm, vias 108 -> 107
- net Net-(Q17-S): track 0.00 -> 4.61 mm
- net Net-(U7-PA4): track 0.00 -> 4.56 mm
- net VDD33: track 68.5 -> 65.4 mm, vias 33 -> 32
- net Net-(U7-NRST): track 0.00 -> 2.95 mm
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
Commit message: Update Dragonfly.kicad_pcb
Parts:
- moved C66 21.8 mm to (271.6, 93.0)
- moved C67 21.4 mm to (271.6, 92.0)
- moved C68 21.1 mm to (271.6, 90.7)
- moved C70 21.1 mm to (271.3, 88.9), turned to 90 degrees
- moved C71 19.3 mm to (272.5, 88.9), turned to 90 degrees
- moved C69 19.1 mm to (273.9, 88.9), turned to 90 degrees
- moved R70 14.1 mm to (262.5, 100.7), turned to -90 degrees
- moved R69 12.5 mm to (261.2, 100.7), turned to -90 degrees
- moved R74 11.1 mm to (260.1, 100.7), turned to -90 degrees
- moved C53 1.76 mm to (249.5, 92.1)
- moved R61 1.47 mm to (290.8, 96.0)
- moved D14 0.81 mm to (249.2, 89.8)
- moved R85 0.75 mm to (250.6, 91.9), turned to -90 degrees
- moved C55 0.58 mm to (250.4, 85.0), turned to 180 degrees
- moved C56 0.51 mm to (250.6, 89.8)
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Routing:
- net VOUT: track 6.47 -> 56.1 mm, vias 0 -> 8
- net ESC2_B3: track 11.8 -> 59.7 mm, vias 2 -> 12
- net Net-(J8-Pin_1): track 12.5 -> 51.5 mm, vias 0 -> 5
- net +8V: track 85.3 -> 119.5 mm, vias 9 -> 12
- net ESC2_C4: track 0.00 -> 33.4 mm, vias 0 -> 2
- net ESC2_A3: track 9.43 -> 39.9 mm, vias 0 -> 5
- net Net-(Q14-G): track 0.00 -> 28.2 mm, vias 0 -> 6
- net ESC2_B4: track 0.00 -> 26.3 mm, vias 0 -> 5
- net ESC2_L013: track 0.00 -> 20.1 mm, vias 0 -> 2
- net 5V: track 33.1 -> 52.6 mm, vias 0 -> 12
- net Net-(C70-Pad2): track 35.0 -> 54.2 mm, vias 2 -> 1
- net Net-(U7-PA1): track 6.00 -> 21.5 mm, vias 0 -> 4
- net Net-(Q21-S): track 0.00 -> 14.3 mm, vias 0 -> 2
- net Net-(U9-PA0): track 1.27 -> 14.9 mm, vias 0 -> 3
- net Net-(U7-PA5): track 4.50 -> 17.0 mm, vias 0 -> 2
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
Commit message: Update Dragonfly.kicad_pcb
Parts:
- moved C59 33.1 mm to (280.5, 87.7), turned to 180 degrees
- moved L2 19.7 mm to (264.6, 90.8)
- moved R78 10.0 mm to (242.9, 88.7), turned to 0 degrees
- moved C52 9.62 mm to (242.4, 87.0)
- moved C50 9.62 mm to (243.4, 87.0)
- moved R87 9.53 mm to (259.2, 101.0), turned to 90 degrees
- moved C32 7.93 mm to (242.9, 112.0)
- moved C34 7.93 mm to (241.9, 112.1)
- moved R74 4.45 mm to (255.8, 99.5), turned to 0 degrees
- moved R75 1.70 mm to (249.6, 102.8), turned to -90 degrees
- moved R68 1.57 mm to (249.9, 100.9)
- moved R88 0.85 mm to (257.5, 97.8), turned to 90 degrees
- moved C35 0.64 mm to (248.8, 123.6)
- moved C48 0.53 mm to (240.7, 100.5)
- moved R28 0.52 mm to (250.1, 113.8)
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Routing:
- net +8V: track 119.5 -> 190.9 mm, vias 12 -> 26
- net ESC2_B2: track 0.00 -> 48.7 mm, vias 0 -> 12
- net ESC2_A2: track 0.00 -> 40.0 mm, vias 0 -> 2
- net BOOT0: track 45.6 -> 82.1 mm, vias 1 -> 3
- net Net-(U9-PA1): track 0.00 -> 36.1 mm, vias 0 -> 11
- net Net-(U5-PA1): track 0.00 -> 32.4 mm, vias 0 -> 4
- net ESC2_C2: track 0.00 -> 27.7 mm, vias 0 -> 4
- net ESC2_L012: track 0.00 -> 19.2 mm, vias 0 -> 7
- net Net-(Q9-S): track 0.00 -> 19.0 mm
- net SWCLK2: track 0.00 -> 18.7 mm, vias 0 -> 2
- net Net-(U5-PA5): track 0.00 -> 17.2 mm, vias 0 -> 2
- net Net-(Q8-G): track 0.00 -> 16.8 mm, vias 0 -> 2
- net Net-(U9-PA4): track 0.00 -> 16.6 mm, vias 0 -> 4
- net Net-(D15-K): track 36.1 -> 20.1 mm
- net SWDIO2: track 0.00 -> 14.9 mm, vias 0 -> 2
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