File: PCB/Dragonfly/.history/Dragonfly.kicad_pcb (KiCad board)
At the start: 4 copper layers, 66 x 58.8 mm, 242 parts, among them J1 Conn_01x04_Pin, J7 XT60PW-M, J8 CAM VIN, J9 VOUT, Q1 Q_NMOS_GDS, Q10 Q_NMOS_GDS, Q11 Q_NMOS_GDS, Q12 Q_NMOS_GDS, Q13 Q_NMOS_GDS, Q14 Q_NMOS_GDS, Q15 Q_NMOS_GDS, Q16 Q_NMOS_GDS, Q17 Q_NMOS_GDS, Q18 Q_NMOS_GDS, Q19 Q_NMOS_GDS, Q2 Q_NMOS_GDS, Q20 Q_NMOS_GDS, Q21 Q_NMOS_GDS, Q22 Q_NMOS_GDS, Q23 Q_NMOS_GDS, Q24 Q_NMOS_GDS, Q3 Q_NMOS_GDS, Q4 Q_NMOS_GDS, Q5 Q_NMOS_GDS, Q6 Q_NMOS_GDS, Q7 Q_NMOS_GDS, Q8 Q_NMOS_GDS, Q9 Q_NMOS_GDS, SW1 SW_SPST, SW2 SW_SPST, U1 STM32F405RGTx, U10 FD6288Q, U11 TPS5430DDA, U12 AMS1117-3.3, U13 L78L08_SO8, U14 AT7456E, U15 BMP280, U2 ICM-20602, U3 AT32F421G8U7, U4 FD6288Q, U5 AT32F421G8U7, U6 FD6288Q, U7 AT32F421G8U7, U8 FD6288Q, U9 AT32F421G8U7, X1 TSX-3225, Y1 27MHZ

Commit message: Update Dragonfly.kicad_pcb
Parts:
- moved C21 8.75 mm to (294.2, 128.7)
- moved C22 8.75 mm to (295.2, 128.7)
Routing:
- net GND: track 133.8 -> 133.2 mm, vias 109 -> 110
- net VDD33: track 68.0 -> 67.6 mm, vias 39 -> 38
Changed lines of the file:
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@@
 	(footprint "Capacitor_SMD:C_0402_1005Metric"
 		(layer "B.Cu")
-		(at 292.5375 120.36 90)
+		(at 295.21 128.69 90)
 		(descr "Capacitor SMD 0402 (1005 Metric), square (rectangular) end terminal, IPC-7351 nominal, (Body size source: IPC-SM-782 page 76, https://www.pcb-3d.com/wordpress/wp-content/uploads/ipc-sm-782a_amendment_1_and_2.pdf)")
 		(tags "capacitor")
@@
 			(net "VDD33")
 			(pintype "passive")
-			(clearance 0.1)
 		)
 		(pad "2" smd roundrect
@@
 			(net "GND")
 			(pintype "passive")
-			(clearance 0.1)
 		)
 		(embedded_fonts no)
@@
 			(pinfunction "VDD_17")
 			(pintype "input")
-			(clearance 0.1)
 		)
 		(pad "18" smd rect
@@
 			(pinfunction "PA8_18")
 			(pintype "output")
-			(clearance 0.1)
 		)
 		(pad "19" smd rect
@@
 	(footprint "Capacitor_SMD:C_0402_1005Metric"
 		(layer "B.Cu")
-		(at 291.5225 120.36 -90)
+		(at 294.195 128.69 -90)
 		(descr "Capacitor SMD 0402 (1005 Metric), square (rectangular) end terminal, IPC-7351 nominal, (Body size source: IPC-SM-782 page 76, https://www.pcb-3d.com/wordpress/wp-content/uploads/ipc-sm-782a_amendment_1_and_2.pdf)")
 		(tags "capacitor")
@@
 			(net "GND")
 			(pintype "passive")
-			(clearance 0.1)
 		)
 		(pad "2" smd roundrect
@@
 			(net "VDD33")
 			(pintype "passive")
-			(clearance 0.1)
 		)
 		(embedded_fonts no)
@@
 	)
 	(via
-		(at 292.5375 119.88)
+		(at 295.21 128.21)
 		(size 0.4)
 		(drill 0.2)
@@
 	)
 	(via
+		(at 246.65 97.793028)
+		(size 0.4)
+		(drill 0.2)
+		(layers "F.Cu" "B.Cu")
+		(net "GND")
+	)
+	(via
 		(at 261.5 114.6)
 		(size 0.4)
@@
 	)
 	(via
-		(at 291.03 115.46)
+		(at 291.375 116.02)
 		(size 0.4)
 		(drill 0.2)
@@
 	)
 	(segment
+		(start 292.2 116.845)
+		(end 291.375 116.02)
+		(width 0.2)
+		(layer "B.Cu")
+		(net "GND")
+	)
+	(segment
 		(start 279.87 88.57)
 		(end 280.1 88.8)
@@
 	)
 	(segment
+		(start 246.65 97.74)
+		(end 246.65 97.793028)
+		(width 0.2)
+		(layer "B.Cu")
+		(net "GND")
+	)
+	(segment
 		(start 246.77 125.47)
 		(end 246.77 125.8)
@@
 	)
 	(segment
+		(start 292.2 118.07)
+		(end 292.2 116.845)
+		(width 0.2)
+		(layer "B.Cu")
+		(net "GND")
+	)
+	(segment
 		(start 241.92 112.54)
 		(end 241.78 112.54)
@@
 	)
 	(segment
-		(start 291.03 115.675)
-		(end 292.2 116.845)
-		(width 0.2)
-		(layer "B.Cu")
-		(net "GND")
-	)
-	(segment
 		(start 259.535 131.375)
 		(end 259.535 131.665)
@@
 	)
 	(segment
-		(start 292.2 116.845)
-		(end 292.2 118.07)
-		(width 0.2)
-		(layer "B.Cu")
-		(net "GND")
-	)
-	(segment
 		(start 290.665 99.665)
 		(end 291.49 100.49)
@@
 	)
 	(segment
-		(start 291.03 115.46)
-		(end 291.03 115.675)
-		(width 0.2)
-		(layer "B.Cu")
-		(net "GND")
-	)
-	(segment
 		(start 288.97 84.22)
 		(end 288.45 84.22)
@@
 	)
 	(segment
-		(start 292.5375 119.88)
-		(end 291.5225 119.88)
+		(start 295.21 128.21)
+		(end 294.195 128.21)
 		(width 0.2)
 		(layer "B.Cu")
@@
 	)
 	(segment
-		(start 291.3025 119.69)
-		(end 291.4925 119.69)
+		(start 293.975 128.02)
+		(end 294.165 128.02)
 		(width 0.2)
 		(layer "B.Cu")
@@
 	)
 	(via
-		(at 292.14 118.79)
-		(size 0.4)
-		(drill 0.2)
-		(layers "F.Cu" "B.Cu")
-		(net "VDD33")
-	)
-	(via
-		(at 246.65 97.793028)
-		(size 0.4)
-		(drill 0.2)
-		(layers "F.Cu" "B.Cu")
-		(net "VDD33")
-	)
-	(via
 		(at 271.35 117.5)
 		(size 0.6)
@@
 	)
 	(via
-		(at 292.5375 120.84)
+		(at 291.71 117.52)
+		(size 0.3)
+		(drill 0.15)
+		(layers "F.Cu" "B.Cu")
+		(free yes)
+		(net "VDD33")
+	)
+	(via
+		(at 295.21 129.17)
 		(size 0.4)
 		(drill 0.2)
@@
 	)
 	(segment
-		(start 291.8 118.07)
-		(end 291.8 118.45)
-		(width 0.2)
-		(layer "B.Cu")
-		(net "VDD33")
-	)
-	(segment
-		(start 246.65 97.74)
-		(end 246.65 97.793028)
+		(start 295.08 95.67)
+		(end 294.1 95.67)
 		(width 0.2)
 		(layer "B.Cu")
@@
 	)
 	(segment
-		(start 295.08 95.67)
-		(end 294.1 95.67)
+		(start 291.8 117.61)
+		(end 291.71 117.52)
 		(width 0.2)
 		(layer "B.Cu")
@@
 	)
 	(segment
+		(start 291.8 118.07)
+		(end 291.8 117.61)
+		(width 0.2)
+		(layer "B.Cu")
+		(net "VDD33")
+	)
+	(segment
 		(start 269.08 109.22)
 		(end 269.38 108.92)
@@
 	)
 	(segment
-		(start 291.5225 120.84)
-		(end 292.5375 120.84)
+		(start 294.195 129.17)
+		(end 295.21 129.17)
 		(width 0.2)
 		(layer "B.Cu")
@@
 	)
 	(segment
-		(start 291.8 118.45)
-		(end 292.14 118.79)
-		(width 0.2)
-		(layer "B.Cu")
-		(net "VDD33")
-	)
-	(segment
 		(start 291.47 112.15)
 		(end 291.47 112.874314)
@@
 	)
 	(segment
-		(start 291.522892 121.112892)
-		(end 290.62 120.21)
+		(start 291.72 121.112892)
+		(end 292.138554 121.531446)
 		(width 0.2)
 		(layer "F.Cu")
@@
 	(segment
 		(start 290.62 120.21)
-		(end 290.62 119.153554)
+		(end 291.522892 121.112892)
 		(width 0.2)
 		(layer "F.Cu")
@@
 	)
 	(segment
-		(start 291.72 121.112892)
-		(end 291.522892 121.112892)
+		(start 291.522892 121.112892)
+		(end 291.72 121.112892)
 		(width 0.2)
 		(layer "F.Cu")
@@
 	)
 	(segment
-		(start 292.19645 121.589342)
-		(end 291.72 121.112892)
+		(start 290.62 119.153554)
+		(end 290.62 120.21)
 		(width 0.2)
 		(layer "F.Cu")
@@
 	)
 	(via
-		(at 292.19645 121.589342)
+		(at 292.138554 121.531446)
 		(size 0.4)
 		(drill 0.2)
@@
 	)
 	(segment
+		(start 292.138554 121.531446)
+		(end 292.138554 121.568554)
+		(width 0.2)
+		(layer "B.Cu")
+		(net "HI21")
+	)
+	(segment
 		(start 290.62 119.113457)
 		(end 291 118.733457)
@@
 	)
 	(segment
-		(start 292.19645 121.589342)
-		(end 292.19645 121.62645)
+		(start 292.138554 121.568554)
+		(end 292.425597 121.855597)
 		(width 0.2)
 		(layer "B.Cu")
@@
 	)
 	(segment
-		(start 292.19645 121.62645)
-		(end 292.425597 121.855597)
+		(start 291.65 119)
+		(end 291.4 118.75)
 		(width 0.2)
 		(layer "B.Cu")
-		(net "HI21")
+		(net "HI31")
 	)
 	(segment
-		(start 291.4 118.07)
-		(end 291.4 119.09)
+		(start 292.971134 119)
+		(end 291.65 119)
 		(width 0.2)
 		(layer "B.Cu")
@@
 	)
 	(segment
-		(start 291.4 119.09)
-		(end 291.6 119.29)
+		(start 293.12 119.148866)
+		(end 292.971134 119)
 		(width 0.2)
 		(layer "B.Cu")
@@
 	)
 	(segment
-		(start 293 119.29)
-		(end 293.12 119.41)
-		(width 0.2)
-		(layer "B.Cu")
-		(net "HI31")
-	)
-	(segment
-		(start 291.6 119.29)
-		(end 293 119.29)
+		(start 291.4 118.75)
+		(end 291.4 118.12)
 		(width 0.2)
 		(layer "B.Cu")
@@
 	(segment
 		(start 293.12 122.268705)
-		(end 293.12 119.41)
+		(end 293.12 119.148866)
 		(width 0.2)
 		(layer "B.Cu")

Commit message: Update Dragonfly.kicad_pcb
Parts:
- added REF**: MountingHole_2.2mm_M2_DIN965_Pad_TopBottom, MountingHole:MountingHole_2.2mm_M2_DIN965_Pad_TopBottom, F.Cu at (238.5, 82.3)
- added REF**: MountingHole_2.2mm_M2_DIN965_Pad_TopBottom, MountingHole:MountingHole_2.2mm_M2_DIN965_Pad_TopBottom, F.Cu at (238.1, 134.9)
- added REF**: MountingHole_2.2mm_M2_DIN965_Pad_TopBottom, MountingHole:MountingHole_2.2mm_M2_DIN965_Pad_TopBottom, F.Cu at (298.2, 82.6)
- added REF**: MountingHole_2.2mm_M2_DIN965_Pad_TopBottom, MountingHole:MountingHole_2.2mm_M2_DIN965_Pad_TopBottom, F.Cu at (297.8, 135.3)
- moved C21 0.21 mm to (294.0, 128.6)
- moved C22 0.21 mm to (295.0, 128.6)
Connections:
- C18 pad 1: VDD33 -> VDD
- C19 pad 1: VDD33 -> VDD
- C20 pad 1: VDD33 -> VDD
- U2 pad 1: VDD33 -> VDD
- U2 pad 16: VDD33 -> VDD
Routing:
- net VDD: track 0.00 -> 9.60 mm, vias 0 -> 2
- net VDD33: track 67.6 -> 62.8 mm, vias 38 -> 35
- net VIN: track 257.2 -> 254.8 mm
- net ESC2_L014: track 5.03 -> 3.42 mm, vias 3 -> 2
- net GND: track 133.2 -> 134.7 mm
- net 5V: track 52.6 -> 51.4 mm, vias 12 -> 11
- net HI31: track 5.91 -> 4.98 mm
- net ESC2_B1: track 37.7 -> 38.5 mm
- net VOUT: track 50.8 -> 50.1 mm
- net ESC2_B3: track 59.3 -> 58.7 mm
- net Net-(U7-BOOT0): track 7.55 -> 6.96 mm
- net ESC2_C3: track 31.4 -> 30.9 mm
- net BOOT0: track 82.1 -> 81.6 mm, vias 3 -> 2
- net ESC2_B4: vias 7 -> 6
- net +8V: track 190.9 -> 191.0 mm, vias 26 -> 25
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